Commit message: Add gazebo argument to realsense urdf

File: eager_sensors/eager_sensor_realsense/urdf/realsense.urdf.xacro (robot description, xacro)
@@ -2,6 +2,6 @@
   <!-- import the camera -->
   <xacro:include filename="$(find realsense2_description)/urdf/_d435.urdf.xacro" />
-  <xacro:include filename="$(find eager_sensor_realsense)/urdf/camera.gazebo.xacro" />
   <!-- camera params-->
+  <xacro:arg name="gazebo"                  default="false"/>
   <xacro:arg name="camera_name"             default="camera"/>
   <xacro:arg name="camera_origin_xyz"       default="0 0 0"/>
@@ -12,4 +12,5 @@
   <xacro:arg name="color_width"             default="1920"/>
   <xacro:arg name="color_height"            default="1080"/>
+  <xacro:property name="load_gazebo" value="$(arg gazebo)"/>
   <link name="world"/>
   <!-- camera -->
@@ -17,10 +18,13 @@
     <origin xyz="$(arg camera_origin_xyz)" rpy="$(arg camera_origin_rpy)" />
   </xacro:sensor_d435>
-  <xacro:my_camera
-    name="$(arg camera_name)"
-    depth_width="$(arg depth_width)"
-    depth_height="$(arg depth_height)"
-    color_width="$(arg color_width)"
-    color_height="$(arg color_height)"
-  />
+  <xacro:if value="${load_gazebo}">
+    <xacro:include filename="$(find eager_sensor_realsense)/urdf/camera.gazebo.xacro" />
+    <xacro:my_camera
+      name="$(arg camera_name)"
+      depth_width="$(arg depth_width)"
+      depth_height="$(arg depth_height)"
+      color_width="$(arg color_width)"
+      color_height="$(arg color_height)"
+    />
+  </xacro:if>
 </robot>
