Commit message: Create urdf that is compatible with pybullet and gazebo

File: eager_sensors/eager_sensor_multisense_s21/urdf/multisense_s21.urdf.xacro (robot description, xacro)
@@ -1,7 +1,13 @@
 <robot name="multisense" xmlns:xacro="http://ros.org/wiki/xacro">
+  <xacro:arg name="gazebo"                  default="false"/>
+  <xacro:property name="load_gazebo" value="$(arg gazebo)"/>
   <!-- import the camera -->
-  <xacro:include filename="$(find eager_sensor_multisense_s21)/urdf/camera.gazebo.xacro" />
+  <xacro:include filename="$(find eager_sensor_multisense_s21)/urdf/s21.urdf.xacro" />
   <link name="world"/>
   <!-- camera -->
-  <xacro:my_camera parent="world"/>
+  <xacro:sensor_s21 parent="world"/>
+  <xacro:if value="${load_gazebo}">
+    <xacro:include filename="$(find eager_sensor_multisense_s21)/urdf/s21.gazebo.xacro" />
+    <xacro:s21_gazebo/>
+  </xacro:if>
 </robot>

File: eager_sensors/eager_sensor_multisense_s21/urdf/s21.gazebo.xacro (robot description, xacro)
@@ -1,85 +1,5 @@
 <?xml version="1.0"?>
 <robot xmlns:xacro="http://www.ros.org/wiki/xacro">
-  <xacro:macro name="my_camera" params="parent">
-    <joint name="dummy_joint" type="fixed">
-        <origin xyz="0.0 0.0 0.0"/>
-        <parent link="${parent}"/>
-        <child link="head"/>
-    </joint>
-    <link name="head">
-        <inertial>
-          <origin xyz="-0.075493 3.3383E-05 0.02774" rpy="0 0 0" />
-          <mass value="1.4199" />
-          <inertia iyy="0.0041178" ixy="-1.5797E-06" iyz="-6.8415E-07" ixx="0.0039688" ixz="-0.00089293" izz="0.0035243" />
-        </inertial>
-        <visual>
-          <origin xyz="0 0 0" rpy="1.57079632679 0 1.57079632679" />
-          <geometry>
-              <mesh filename="package://eager_sensor_multisense_s21/meshes/multisense_s21.dae"/>
-          </geometry>
-          <material name="">
-              <color rgba="0.9098 0.44314 0.031373 1" />
-          </material>
-        </visual>
-        <collision>
-          <origin xyz="-0.0503 0 -0.00195" rpy="0 0 0" />
-          <geometry>
-            <box size="0.1311 0.12 0.0591"/>
-          </geometry>
-        </collision>
-    </link>
-    <!-- Note the origin of model is 37.3854mm from the rear mounting plane
-         in the x axis -->
-    <joint name="left_camera_joint" type="fixed">
-        <origin xyz="0.07 0.105 0.0"/>
-        <parent link="head"/>
-        <child link="left_camera_frame"/>
-    </joint>
-    <link name="left_camera_frame"/>
-    <joint name="right_camera_joint" type="fixed">
-        <origin xyz="0.07 -0.105 0.0"/>
-        <parent link="head"/>
-        <child link="right_camera_frame"/>
-    </joint>
-    <link name="right_camera_frame"/>
-    <joint name="left_camera_optical_joint" type="fixed">
-        <origin xyz="0.0052046 0 0" rpy="-1.57079632679 0.0 -1.57079632679"/>
-        <parent link="left_camera_frame"/>
-        <child link="left_camera_optical_frame"/>
-    </joint>
-    <link name="left_camera_optical_frame"/>
-    <joint name="right_camera_optical_joint" type="fixed">
-        <origin xyz="0.0052046 0 0" rpy="-1.57079632679 0.0 -1.57079632679"/>
-        <parent link="right_camera_frame"/>
-        <child link="right_camera_optical_frame"/>
-    </joint>
-    <link name="right_camera_optical_frame"/>
-    <joint name="top_left_rear_mount_joint" type="fixed">
-        <origin xyz="-0.0373854 0.1 0.014" rpy="0 0 3.14159"/>
-        <parent link="head"/>
-        <child link="top_left_rear_mount"/>
-    </joint>
-    <link name="top_left_rear_mount"/>
-    <!--Note the locations of the accel/mag and gyro differ from those shown
-        in CAD. The S21 firmware switches axis on the accel/mag and gyro to
-        match the S7/S7S/SL MultiSense configurations -->
-    <joint name="accel_joint" type="fixed">
-        <origin xyz="0.0045 0.029 -0.0135" rpy="0.0 1.57079632679 0.0"/>
-        <parent link="head"/>
-        <child link="accel"/>
-    </joint>
-    <link name="accel"/>
-    <joint name="mag_joint" type="fixed">
-        <origin xyz="0.0045 0.029 -0.0135" rpy="0.0 1.57079632679 0.0"/>
-        <parent link="head"/>
-        <child link="mag"/>
-    </joint>
-    <link name="mag"/>
-    <joint name="gyro_joint" type="fixed">
-        <origin xyz="-0.00219539 0.03758 -0.014" rpy="-1.57079632679 0 -1.57079632679"/>
-        <parent link="head"/>
-        <child link="gyro"/>
-    </joint>
-    <link name="gyro"/>
+  <xacro:macro name="s21_gazebo">
     <gazebo reference="head">
       <material>Gazebo/DarkGrey </material>
